File: pcb/relai-lit-electrique.brd (EAGLE design)
At the start: 58 x 80 mm, 24 parts, among them K1 DSP1.1A, Q3 2N5484, Q4 2N5484, X1 DSP-3, X2 DSP-3

Commit message: update
Parts:
- removed C3: 100n, rcl:C025-024X044
Connections:
- net +3V3: no longer C3.1
- net GND: no longer C3.2
Routing:
- net N$7: track 35.0 -> 0.00 mm
- net GND: track 151.9 -> 146.9 mm
- net +3V3: track 179.4 -> 178.8 mm
Changed lines of the file:
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@@
 </autorouter>
 <elements>
-<element name="C3" library="rcl" package="C025-024X044" value="100n" x="3.81" y="46.355" rot="R180"/>
 <element name="D1" library="diode" package="DO41-10" value="1N4004" x="40.005" y="39.37" rot="R180"/>
 <element name="D2" library="diode" package="DO41-10" value="1N4004" x="40.005" y="43.18" rot="R180"/>
@@
 <contactref element="R4" pad="1"/>
 <contactref element="R5" pad="1"/>
-<contactref element="IC2" pad="V-"/>
-<contactref element="C3" pad="2"/>
 <contactref element="LED1" pad="K"/>
 <contactref element="MOD1" pad="GND"/>
@@
 <contactref element="Q4" pad="2"/>
 <contactref element="OK1" pad="3"/>
-<contactref element="C1" pad="-"/>
 <wire x1="40.7778" y1="9.1542" x2="34.9524" y2="3.3288" width="0.6096" layer="16"/>
 <wire x1="40.7778" y1="24.4112" x2="40.7778" y2="9.1542" width="0.6096" layer="16"/>
@@
 <wire x1="16.3666" y1="14.1474" x2="13.5926" y2="16.9214" width="0.6096" layer="16"/>
 <wire x1="13.5926" y1="22.7468" x2="13.335" y2="22.86" width="0.6096" layer="16"/>
-<wire x1="16.3666" y1="14.1474" x2="16.383" y2="13.97" width="0.6096" layer="16"/>
 <wire x1="12.483" y1="16.0892" x2="5.8254" y2="16.0892" width="0.6096" layer="16"/>
 <wire x1="13.3152" y1="16.9214" x2="12.483" y2="16.0892" width="0.6096" layer="16"/>
 <wire x1="5.8254" y1="16.0892" x2="5.715" y2="15.875" width="0.6096" layer="16"/>
 <wire x1="13.3152" y1="16.9214" x2="13.5926" y2="16.9214" width="0.6096" layer="16"/>
-<wire x1="2.4966" y1="50.7642" x2="2.4966" y2="46.6032" width="0.6096" layer="16"/>
-<wire x1="2.4966" y1="46.6032" x2="2.54" y2="46.355" width="0.6096" layer="16"/>
-<wire x1="2.4966" y1="50.7642" x2="2.54" y2="50.8" width="0.6096" layer="16"/>
 <wire x1="38.5586" y1="29.4044" x2="33.8428" y2="29.4044" width="0.6096" layer="16"/>
 <wire x1="39.6682" y1="30.514" x2="38.5586" y2="29.4044" width="0.6096" layer="16"/>
@@
 <wire x1="26.9078" y1="36.062" x2="26.9078" y2="37.449" width="0.6096" layer="16"/>
 <wire x1="33.5654" y1="29.4044" x2="26.9078" y2="36.062" width="0.6096" layer="16"/>
-<wire x1="2.774" y1="51.0416" x2="2.54" y2="50.8" width="0.6096" layer="16"/>
 <wire x1="33.5654" y1="29.4044" x2="33.655" y2="29.21" width="0.6096" layer="16"/>
 <wire x1="13.5926" y1="31.6236" x2="13.5926" y2="23.0242" width="0.6096" layer="16"/>
@@
 <wire x1="43.8292" y1="27.4626" x2="43.815" y2="27.305" width="0.6096" layer="16"/>
 <wire x1="42.7196" y1="33.8428" x2="42.545" y2="33.655" width="0.6096" layer="16"/>
+<contactref element="C1" pad="-"/>
+<contactref element="IC2" pad="V-"/>
+<wire x1="2.774" y1="51.0416" x2="2.54" y2="50.8" width="0" layer="19" extent="16-16"/>
+<wire x1="16.383" y1="13.97" x2="16.3666" y2="14.1474" width="0" layer="19" extent="16-16"/>
 </signal>
 <signal name="PHASE" class="1">
@@
 <contactref element="K1" pad="P$15"/>
 <contactref element="D1" pad="C"/>
-<contactref element="D2" pad="C"/>
-<contactref element="K1" pad="P$16"/>
 <contactref element="IC2" pad="V+"/>
-<contactref element="C3" pad="1"/>
 <contactref element="MOD1" pad="3V3"/>
 <contactref element="R1" pad="2"/>
@@
 <wire x1="5.2706" y1="46.3258" x2="5.8254" y2="45.771" width="0.6096" layer="16"/>
 <wire x1="10.5412" y1="45.771" x2="10.795" y2="45.72" width="0.6096" layer="16"/>
-<wire x1="5.2706" y1="46.3258" x2="5.08" y2="46.355" width="0.6096" layer="16"/>
 <wire x1="7.7672" y1="50.7642" x2="7.7672" y2="46.0484" width="0.6096" layer="16"/>
 <wire x1="7.7672" y1="46.0484" x2="7.7672" y2="45.771" width="0.6096" layer="16"/>
@@
 <wire x1="45.2162" y1="42.997" x2="45.2162" y2="39.3908" width="0.6096" layer="16"/>
 <wire x1="45.2162" y1="39.3908" x2="45.085" y2="39.37" width="0.6096" layer="16"/>
-<wire x1="45.2162" y1="42.997" x2="45.085" y2="43.18" width="0.6096" layer="16"/>
 <wire x1="45.771" y1="53.8156" x2="45.771" y2="51.5964" width="0.6096" layer="16"/>
-<wire x1="45.771" y1="51.5964" x2="45.72" y2="51.435" width="0.6096" layer="16"/>
 <wire x1="45.771" y1="53.8156" x2="45.72" y2="53.975" width="0.6096" layer="16"/>
-<wire x1="45.2162" y1="51.0416" x2="45.2162" y2="43.2744" width="0.6096" layer="16"/>
-<wire x1="45.4936" y1="51.319" x2="45.2162" y2="51.0416" width="0.6096" layer="16"/>
-<wire x1="45.2162" y1="43.2744" x2="45.085" y2="43.18" width="0.6096" layer="16"/>
-<wire x1="45.4936" y1="51.319" x2="45.72" y2="51.435" width="0.6096" layer="16"/>
 <wire x1="45.2162" y1="33.0106" x2="45.2162" y2="39.1134" width="0.6096" layer="16"/>
 <wire x1="46.0484" y1="32.1784" x2="45.2162" y2="33.0106" width="0.6096" layer="16"/>
@@
 <wire x1="45.2162" y1="39.1134" x2="45.085" y2="39.37" width="0.6096" layer="16"/>
 <wire x1="25.5208" y1="10.2638" x2="25.3821" y2="10.4025" width="0.6096" layer="16"/>
+<contactref element="D2" pad="C"/>
+<contactref element="K1" pad="P$16"/>
+<wire x1="45.2162" y1="51.0416" x2="45.2162" y2="43.2744" width="0.6096" layer="16"/>
+<wire x1="45.4936" y1="51.319" x2="45.2162" y2="51.0416" width="0.6096" layer="16"/>
+<wire x1="45.2162" y1="43.2744" x2="45.085" y2="43.18" width="0.6096" layer="16"/>
+<wire x1="45.4936" y1="51.319" x2="45.72" y2="51.435" width="0.6096" layer="16"/>
+<wire x1="45.72" y1="51.435" x2="45.771" y2="51.5964" width="0" layer="19" extent="16-16"/>
+<wire x1="45.2162" y1="42.997" x2="45.085" y2="43.18" width="0" layer="19" extent="16-16"/>
 </signal>
 <signal name="N$8" class="1">
@@
 <wire x1="5.8254" y1="8.0446" x2="5.715" y2="8.255" width="0.6096" layer="16"/>
 <wire x1="25.2434" y1="3.8836" x2="25.32" y2="3.81" width="0.6096" layer="16"/>
-</signal>
-<signal name="N$16">
-<contactref element="OK1" pad="4"/>
-<contactref element="R1" pad="1"/>
-<contactref element="C2" pad="1"/>
-<wire x1="3.3288" y1="18.8632" x2="3.3288" y2="16.0892" width="0.6096" layer="16"/>
-<wire x1="3.3288" y1="16.0892" x2="3.175" y2="15.875" width="0.6096" layer="16"/>
-<wire x1="3.3288" y1="18.8632" x2="3.175" y2="19.05" width="0.6096" layer="16"/>
-<wire x1="26.0756" y1="15.257" x2="23.579" y2="17.7536" width="0.6096" layer="16"/>
-<wire x1="26.0756" y1="12.7604" x2="26.0756" y2="15.257" width="0.6096" layer="16"/>
-<wire x1="24.4112" y1="11.096" x2="26.0756" y2="12.7604" width="0.6096" layer="16"/>
-<wire x1="8.0446" y1="11.096" x2="24.4112" y2="11.096" width="0.6096" layer="16"/>
-<wire x1="3.3288" y1="15.8118" x2="8.0446" y2="11.096" width="0.6096" layer="16"/>
-<wire x1="23.579" y1="17.7536" x2="23.495" y2="17.78" width="0.6096" layer="16"/>
-<wire x1="3.3288" y1="15.8118" x2="3.175" y2="15.875" width="0.6096" layer="16"/>
 </signal>
 <signal name="N$4">
@@
 <wire x1="5.548" y1="19.1406" x2="5.715" y2="19.05" width="0.6096" layer="16"/>
 </signal>
+<signal name="N$7">
+<contactref element="R1" pad="1"/>
+<contactref element="C2" pad="1"/>
+<contactref element="OK1" pad="4"/>
+<wire x1="3.175" y1="19.05" x2="23.495" y2="17.78" width="0" layer="19" extent="1-1"/>
+<wire x1="3.175" y1="15.875" x2="3.175" y2="19.05" width="0" layer="19" extent="1-1"/>
+</signal>
 </signals>
